File: Adapter-IO4-Grove.brd (EAGLE design)
At the start: 50 x 50 mm, 7 parts, among them J1 CONNECTOR-GROVE-4P-2.0-347013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, J2 CONNECTOR-GROVE-4P-2.0-347013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, J3 CONNECTOR-GROVE-4P-2.0-347013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, J4 CONNECTOR-GROVE-4P-2.0-347013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

Commit message: added values for connectors
Parts:
- J-IO4: value (none) -> RJ12/6
Changed lines of the file:
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@@
 <element name="LOGO1" library="SPCoast" package="OSHW-LOGO-L" value="DOC-OSHW-LOGO-L" x="5.08" y="44.45"/>
 <element name="U$1" library="SPCoast" package="BOARD-SEEED5X5" value="BOARD50X50" x="0" y="0"/>
-<element name="J-IO4" library="SPCoast" package="RJ25-INVERTED" value="" x="7.62" y="25.4" rot="R270"/>
+<element name="J-IO4" library="SPCoast" package="RJ25-INVERTED" value="RJ12/6" x="7.62" y="25.4" rot="R270"/>
 <element name="J1" library="SPCoast" package="4P-2.0" value="CONNECTOR-GROVE-4P-2.0-3470130P1" x="25.4" y="15.24" smashed="yes" rot="R90">
 <attribute name="NAME" x="22.86" y="13.335" size="0.889" layer="25" font="vector" ratio="11" rot="R90"/>

Commit message: normalized values
Parts:
- J1, J2, J3, J4: value CONNECTOR-GROVE-4P-2.0-3470130P1 -> 2mm
- LOGO1: value DOC-OSHW-LOGO-L -> OSHW
- U$1: value BOARD50X50 -> BOARD
Changed lines of the file:
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@@
 </autorouter>
 <elements>
-<element name="LOGO1" library="SPCoast" package="OSHW-LOGO-L" value="DOC-OSHW-LOGO-L" x="5.08" y="44.45"/>
-<element name="U$1" library="SPCoast" package="BOARD-SEEED5X5" value="BOARD50X50" x="0" y="0"/>
+<element name="LOGO1" library="SPCoast" package="OSHW-LOGO-L" value="OSHW" x="5.08" y="44.45"/>
+<element name="U$1" library="SPCoast" package="BOARD-SEEED5X5" value="BOARD" x="0" y="0"/>
 <element name="J-IO4" library="SPCoast" package="RJ25-INVERTED" value="RJ12/6" x="7.62" y="25.4" rot="R270"/>
-<element name="J1" library="SPCoast" package="4P-2.0" value="CONNECTOR-GROVE-4P-2.0-3470130P1" x="25.4" y="15.24" smashed="yes" rot="R90">
+<element name="J1" library="SPCoast" package="4P-2.0" value="2mm" x="25.4" y="15.24" smashed="yes" rot="R90">
 <attribute name="NAME" x="22.86" y="13.335" size="0.889" layer="25" font="vector" ratio="11" rot="R90"/>
 </element>
-<element name="J2" library="SPCoast" package="4P-2.0" value="CONNECTOR-GROVE-4P-2.0-3470130P1" x="25.4" y="35.56" smashed="yes" rot="R90">
+<element name="J2" library="SPCoast" package="4P-2.0" value="2mm" x="25.4" y="35.56" smashed="yes" rot="R90">
 <attribute name="NAME" x="22.86" y="33.655" size="0.889" layer="25" font="vector" ratio="11" rot="R90"/>
 </element>
-<element name="J3" library="SPCoast" package="4P-2.0" value="CONNECTOR-GROVE-4P-2.0-3470130P1" x="38.1" y="15.24" smashed="yes" rot="R90">
+<element name="J3" library="SPCoast" package="4P-2.0" value="2mm" x="38.1" y="15.24" smashed="yes" rot="R90">
 <attribute name="NAME" x="35.56" y="13.335" size="0.889" layer="25" font="vector" ratio="11" rot="R90"/>
 </element>
-<element name="J4" library="SPCoast" package="4P-2.0" value="CONNECTOR-GROVE-4P-2.0-3470130P1" x="38.1" y="35.56" smashed="yes" rot="R90">
+<element name="J4" library="SPCoast" package="4P-2.0" value="2mm" x="38.1" y="35.56" smashed="yes" rot="R90">
 <attribute name="NAME" x="35.56" y="33.655" size="0.889" layer="25" font="vector" ratio="11" rot="R90"/>
 </element>
@@
 <wire x1="13.5382" y1="28.4734" x2="38.0746" y2="28.4734" width="0.3048" layer="16"/>
 <wire x1="38.0746" y1="28.4734" x2="38.1" y2="28.448" width="0.3048" layer="16"/>
-<wire x1="38.1" y1="28.448" x2="38.1" y2="32.56" width="0.4064" layer="16"/>
-<wire x1="38.1" y1="14.24" x2="40.275" y2="14.24" width="0.3048" layer="1"/>
+<wire x1="38.1" y1="28.448" x2="37.846" y2="32.56" width="0.4064" layer="16"/>
+<wire x1="38.354" y1="14.24" x2="40.275" y2="14.24" width="0.3048" layer="1"/>
 <wire x1="40.275" y1="14.24" x2="41.275" y2="15.24" width="0.3048" layer="1"/>
 <wire x1="41.275" y1="15.24" x2="41.275" y2="28.4226" width="0.3048" layer="1"/>
@@
 <wire x1="43.18" y1="33.9598" x2="42.5704" y2="34.5694" width="0.3048" layer="16"/>
 <wire x1="42.5704" y1="34.5694" x2="38.1094" y2="34.5694" width="0.3048" layer="16"/>
-<wire x1="38.1094" y1="34.5694" x2="38.1" y2="34.56" width="0.3048" layer="16"/>
+<wire x1="38.1094" y1="34.5694" x2="38.354" y2="34.56" width="0.3048" layer="16"/>
 <wire x1="22.225" y1="21.59" x2="22.225" y2="13.0556" width="0.3048" layer="16"/>
 <wire x1="22.225" y1="13.0556" x2="23.0378" y2="12.2428" width="0.3048" layer="16"/>
 <wire x1="23.0378" y1="12.2428" x2="25.3972" y2="12.2428" width="0.3048" layer="16"/>
-<wire x1="25.3972" y1="12.2428" x2="25.4" y2="12.24" width="0.3048" layer="16"/>
+<wire x1="25.3972" y1="12.2428" x2="25.146" y2="12.24" width="0.3048" layer="16"/>
 </signal>
 <signal name="P2">
@@
 <wire x1="15.875" y1="24.13" x2="25.4" y2="24.13" width="0.3048" layer="16"/>
 <via x="25.4" y="24.13" extent="1-16" drill="0.7" shape="octagon"/>
-<wire x1="25.4" y1="24.13" x2="25.4" y2="32.56" width="0.3048" layer="1"/>
-<wire x1="25.4" y1="14.24" x2="27.575" y2="14.24" width="0.3048" layer="1"/>
+<wire x1="25.4" y1="24.13" x2="25.146" y2="32.56" width="0.3048" layer="1"/>
+<wire x1="25.654" y1="14.24" x2="27.575" y2="14.24" width="0.3048" layer="1"/>
 <wire x1="27.575" y1="14.24" x2="28.575" y2="15.24" width="0.3048" layer="1"/>
 <wire x1="28.575" y1="15.24" x2="28.575" y2="24.13" width="0.3048" layer="1"/>
@@
 <wire x1="28.575" y1="33.7058" x2="27.7114" y2="34.5694" width="0.3048" layer="1"/>
 <wire x1="27.7114" y1="34.5694" x2="25.4094" y2="34.5694" width="0.3048" layer="1"/>
-<wire x1="25.4094" y1="34.5694" x2="25.4" y2="34.56" width="0.3048" layer="1"/>
-<wire x1="38.1" y1="12.24" x2="36.02" y2="12.24" width="0.3048" layer="1"/>
+<wire x1="25.4094" y1="34.5694" x2="25.654" y2="34.56" width="0.3048" layer="1"/>
+<wire x1="37.846" y1="12.24" x2="36.02" y2="12.24" width="0.3048" layer="1"/>
 <wire x1="36.02" y1="12.24" x2="34.925" y2="13.335" width="0.3048" layer="1"/>
 <wire x1="34.925" y1="13.335" x2="34.925" y2="27.305" width="0.3048" layer="1"/>
